File: STM32MP1_TestBoard_RevB/USB_Conn.sch (KiCad schematic (older format))
At the start: 4 parts, among them J13 USB_B_Micro, J8 USB_B_Micro

Commit message: Updated design
- Added Crystal/Oscillators
- Replaced both SDMMC with single SDMMC w/ detect pin
- Added USB Type C for VIN
- Moved SWD pins
- Tidied up silk screen for pin headers J1, J2, J3, J4
- Moved DSI socket
Parts:
- R16, R17: LCSC (none) -> C25077
Changed lines of the file:
@@
 $Descr A4 11693 8268
 encoding utf-8
-Sheet 9 10
+Sheet 9 9
 Title ""
 Date ""
@@
 F 4 "~" H 4625 3200 50  0001 C CNN "Mfr"
 F 5 "~" H 4625 3200 50  0001 C CNN "PartNo"
+F 6 "~" H 4625 3200 50  0001 C CNN "LCSC"
 	1    4625 3200
 	1    0    0    -1
@@
 F 4 "~" H 4650 5050 50  0001 C CNN "Mfr"
 F 5 "~" H 4650 5050 50  0001 C CNN "PartNo"
+F 6 "~" H 4650 5050 50  0001 C CNN "LCSC"
 	1    4650 5050
 	1    0    0    -1
@@
 F 4 "~" H 5200 4850 50  0001 C CNN "Mfr"
 F 5 "~" H 5200 4850 50  0001 C CNN "PartNo"
+F 6 "C25077" H 5200 4850 50  0001 C CNN "LCSC"
 	1    5200 4850
 	0    1    1    0
@@
 F 4 "~" H 4650 5725 50  0001 C CNN "Mfr"
 F 5 "~" H 4650 5725 50  0001 C CNN "PartNo"
+F 6 "C25077" H 4650 5725 50  0001 C CNN "LCSC"
 	1    4650 5725
 	-1   0    0    1

Commit message: completed revb layout
Parts:
- R16, R17: LCSC C25077 -> C25087
Changed lines of the file:
@@
 F 5 "~" H 4625 3200 50  0001 C CNN "PartNo"
 F 6 "~" H 4625 3200 50  0001 C CNN "LCSC"
+F 7 "~" H 4625 3200 50  0001 C CNN "Comment"
+F 8 "~" H 4625 3200 50  0001 C CNN "Mouser"
 	1    4625 3200
 	1    0    0    -1
@@
 F 5 "~" H 4650 5050 50  0001 C CNN "PartNo"
 F 6 "~" H 4650 5050 50  0001 C CNN "LCSC"
+F 7 "~" H 4650 5050 50  0001 C CNN "Comment"
+F 8 "~" H 4650 5050 50  0001 C CNN "Mouser"
 	1    4650 5050
 	1    0    0    -1
@@
 F 4 "~" H 5200 4850 50  0001 C CNN "Mfr"
 F 5 "~" H 5200 4850 50  0001 C CNN "PartNo"
-F 6 "C25077" H 5200 4850 50  0001 C CNN "LCSC"
+F 6 "C25087" H 5200 4850 50  0001 C CNN "LCSC"
+F 7 "~" H 5200 4850 50  0001 C CNN "Comment"
+F 8 "~" H 5200 4850 50  0001 C CNN "Mouser"
 	1    5200 4850
 	0    1    1    0
@@
 F 4 "~" H 4650 5725 50  0001 C CNN "Mfr"
 F 5 "~" H 4650 5725 50  0001 C CNN "PartNo"
-F 6 "C25077" H 4650 5725 50  0001 C CNN "LCSC"
+F 6 "C25087" H 4650 5725 50  0001 C CNN "LCSC"
+F 7 "~" H 4650 5725 50  0001 C CNN "Comment"
+F 8 "~" H 4650 5725 50  0001 C CNN "Mouser"
 	1    4650 5725
 	-1   0    0    1
